Commit message: feat: align URDF physics with ArduPilot servo specs

File: humanoid_skeleton.urdf (robot description, URDF)
Before this commit: robot ardupilot_humanoid, 4 links, 3 joints
Links:
- link l_thigh: mass 1.0 -> 0.5
Joints:
- joint l_hip_pitch: child l_hip_pitch_link -> ; limit lower=-1.5 upper=1.5 effort=10 velocity=1.0 -> lower=-1.571 upper=0.523 effort=20.0 velocity=3.0
- joint l_knee: limit lower=0 upper=2.0 effort=10 velocity=1.0 -> lower=0.0 upper=2.618 effort=15.0 velocity=3.0; origin xyz=0 0 0 rpy=0 0 0 -> xyz=0 0 -0.05 rpy=0 0 0

Commit message: fix: correct joint parent/child link tags

File: humanoid_skeleton.urdf (robot description, URDF)
Before this commit: robot ardupilot_humanoid, 4 links, 3 joints
Links:
- link l_hip_pitch_link: mass None -> 0.1
Joints:
- joint base_to_torso: origin (none) -> xyz=0 0 0 rpy=0 0 0
- joint l_hip_pitch: child  -> l_hip_pitch_link

Commit message: feat: implement mirrored right leg kinematics

File: humanoid_skeleton.urdf (robot description, URDF)
Before this commit: robot ardupilot_humanoid, 4 links, 3 joints
Links:
- added link r_hip_pitch_link, mass 0.1; visual sphere radius=0.03
- added link r_thigh, mass 0.5; visual cylinder length=0.3 radius=0.025
Joints:
- added joint r_hip_pitch: type revolute, parent torso, child r_hip_pitch_link, origin xyz=0 -0.08 0 rpy=0 0 0, axis 0 1 0, limit lower=-1.571 upper=0.523 effort=20.0 velocity=3.0
- added joint r_knee: type revolute, parent r_hip_pitch_link, child , origin xyz=0 0 -0.05 rpy=0 0 0, axis 0 1 0, limit lower=0.0 upper=2.618 effort=15.0 velocity=3.0
