Commit message: refactor: rename URDF to match project naming convention and fix validation path

File: humanoid_proto.urdf (robot description, URDF)
Before this commit: robot ardupilot_humanoid, 8 links, 7 joints
Links:
- link l_foot: mass None -> 0.100
- link l_hip_pitch_link: mass 0.1 -> 0.100
- link l_thigh: mass 0.5 -> 0.500
- link r_foot: mass None -> 0.100
- link r_hip_pitch_link: mass 0.1 -> 0.100
- link r_thigh: mass 0.5 -> 0.500
- link torso: mass 2.5 -> 2.500
Joints:
- joint l_ankle: origin xyz=0 0 -0.31 rpy=0 0 0 -> xyz=0 0 -0.310 rpy=0 0 0
- joint l_hip_pitch: origin xyz=0 0.08 0 rpy=0 0 0 -> xyz=0 0.080 0 rpy=0 0 0
- joint l_knee: origin xyz=0 0 -0.05 rpy=0 0 0 -> xyz=0 0 -0.050 rpy=0 0 0
- joint r_ankle: origin xyz=0 0 -0.31 rpy=0 0 0 -> xyz=0 0 -0.310 rpy=0 0 0
- joint r_hip_pitch: origin xyz=0 -0.08 0 rpy=0 0 0 -> xyz=0 -0.080 0 rpy=0 0 0
- joint r_knee: origin xyz=0 0 -0.05 rpy=0 0 0 -> xyz=0 0 -0.050 rpy=0 0 0

Commit message: fix: clean up duplicate XML tags and fix script pathing

File: humanoid_proto.urdf (robot description, URDF)
Before this commit: robot ardupilot_humanoid, 8 links, 7 joints
Links:
- removed link l_foot
- removed link l_hip_pitch_link
- removed link l_thigh
- removed link r_foot
- removed link r_hip_pitch_link
- removed link r_thigh
Joints:
- removed joint l_ankle
- removed joint l_hip_pitch
- removed joint l_knee
- removed joint r_ankle
- removed joint r_hip_pitch
- removed joint r_knee

Commit message: fix: rename file in workflow and clean up duplicate XML tags

File: humanoid_proto.urdf (robot description, URDF)
Before this commit: robot ardupilot_humanoid, 2 links, 1 joints
Links:
- added link l_foot, mass 0.100; collision box size=0.1 0.08 0.02; visual box size=0.1 0.08 0.02
- added link l_hip_pitch_link, mass 0.100; visual sphere radius=0.03
- added link l_thigh, mass 0.500; visual cylinder length=0.3 radius=0.025
- added link r_foot, mass 0.100; collision box size=0.1 0.08 0.02; visual box size=0.1 0.08 0.02
- added link r_hip_pitch_link, mass 0.100; visual sphere radius=0.03
- added link r_thigh, mass 0.500; visual cylinder length=0.3 radius=0.025
Joints:
- added joint l_ankle: type fixed, parent l_thigh, child l_foot, origin xyz=0 0 -0.310 rpy=0 0 0
- added joint l_hip_pitch: type revolute, parent torso, child l_hip_pitch_link, origin xyz=0 0.080 0 rpy=0 0 0, axis 0 1 0, limit lower=-1.571 upper=0.523 effort=20.0 velocity=3.0
- added joint l_knee: type revolute, parent l_hip_pitch_link, child l_thigh, origin xyz=0 0 -0.050 rpy=0 0 0, axis 0 1 0, limit lower=0.0 upper=2.618 effort=15.0 velocity=3.0
- added joint r_ankle: type fixed, parent r_thigh, child r_foot, origin xyz=0 0 -0.310 rpy=0 0 0
- added joint r_hip_pitch: type revolute, parent torso, child r_hip_pitch_link, origin xyz=0 -0.080 0 rpy=0 0 0, axis 0 1 0, limit lower=-1.571 upper=0.523 effort=20.0 velocity=3.0
- added joint r_knee: type revolute, parent r_hip_pitch_link, child r_thigh, origin xyz=0 0 -0.050 rpy=0 0 0, axis 0 1 0, limit lower=0.0 upper=2.618 effort=15.0 velocity=3.0

Commit message: feat: align imu_link origin for EKF3 compatibility

File: humanoid_proto.urdf (robot description, URDF)
Before this commit: robot ardupilot_humanoid, 8 links, 7 joints
Links:
- added link head, mass 0.2; visual sphere radius=0.05
- added link imu_link, mass 0.01
Joints:
- added joint head_to_imu: type fixed, parent head, child imu_link, origin xyz=0 0 0 rpy=0 0 0
- added joint torso_to_head: type fixed, parent torso, child head, origin xyz=0 0 0.3 rpy=0 0 0

Commit message: fix: physics stability corrections for ArduPilot SITL
- IMU moved to torso CoM, eliminates EKF3 lever-arm error
- Ankle Z offset fixed -0.310 to -0.300m
- Collision geometry added to thighs
- Head inertia corrected 0.0001 to 0.0002 kg*m^2
- Thigh inertia corrected 0.010 to 0.00375 kg*m^2
- calculate_com.py rewritten with world-frame joint transforms
- print_tree.py fixed recursive lookup bug, ASCII safe

File: humanoid_proto.urdf (robot description, URDF)
Before this commit: robot ardupilot_humanoid, 10 links, 9 joints
Links:
- link head: mass 0.2 -> 0.200; geometry collision sphere radius=0.05; visual sphere radius=0.05
- link l_hip_pitch_link: geometry collision sphere radius=0.03; visual sphere radius=0.03
- link l_thigh: geometry collision cylinder length=0.3 radius=0.025; visual cylinder length=0.3 radius=0.025
- link r_hip_pitch_link: geometry collision sphere radius=0.03; visual sphere radius=0.03
- link r_thigh: geometry collision cylinder length=0.3 radius=0.025; visual cylinder length=0.3 radius=0.025
- link torso: geometry collision box size=0.15 0.1 0.3; visual box size=0.15 0.1 0.3
Joints:
- removed joint head_to_imu
- added joint torso_to_imu: type fixed, parent torso, child imu_link, origin xyz=0 0 0.150 rpy=0 0 0
- joint l_ankle: origin xyz=0 0 -0.310 rpy=0 0 0 -> xyz=0 0 -0.300 rpy=0 0 0
- joint r_ankle: origin xyz=0 0 -0.310 rpy=0 0 0 -> xyz=0 0 -0.300 rpy=0 0 0
